File: drive_ctrl.brd (EAGLE design)
At the start: 31 x 34 mm, 24 parts, among them J1 4-PIN_2MM-V, J2 4-PIN_2MM-V, J3 ZEROING_SENSOR, U1 ATTINY84ATTINY84-20PU, U2 DRV8871HSOP-8, U3 AP2210-5KSOT-23-5

Commit message: Added fuse, decoupling capacitors, and changed routing
Parts:
- added F1: 3A, RoboJackets-Fuses:F1206
- added R6: 1k, rcl:R0603
Connections:
- new net 12V_FUSE: C3.1, C4.1, F1.2, U2.5
- net +12V: now also F1.1; no longer C3.1, C4.1, U2.5
- net +5V: now also R6.2
- net RST: now also R6.1
Routing:
- net +12V: track 57.5 -> 48.4 mm, vias 1 -> 0
- net 12V_FUSE: track 0.00 -> 8.81 mm, vias 0 -> 1
- net RST: track 12.2 -> 18.0 mm
- net +5V: track 56.2 -> 60.5 mm, vias 2 -> 3
- net ENC_B: track 28.5 -> 32.4 mm, vias 0 -> 2
- net ENC_A: track 25.9 -> 27.7 mm, vias 0 -> 2
Changed lines of the file:
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@@
 <class number="0" name="default" width="0.2" drill="0">
+</class>
+<class number="1" name="PWR" width="0.6" drill="0">
 </class>
 </classes>
@@
 <attribute name="VALUE" x="5.665" y="14.885" size="1.27" layer="28" rot="MR0"/>
 </element>
+<element name="R6" library="rcl" library_urn="urn:adsk.eagle:library:334" package="R0603" package3d_urn="urn:adsk.eagle:package:23555/3" value="1k" x="8.63" y="10.45" smashed="yes" rot="MR180">
+<attribute name="NAME" x="7.995" y="9.815" size="1.27" layer="26" rot="MR180"/>
+<attribute name="POPULARITY" value="77" x="8.63" y="10.45" size="1" layer="28" font="vector" rot="MR180" display="off"/>
+<attribute name="SPICEPREFIX" value="R" x="8.63" y="10.45" size="1" layer="28" font="vector" rot="MR180" display="off"/>
+<attribute name="VALUE" x="7.995" y="12.355" size="1.27" layer="28" rot="MR180"/>
+</element>
+<element name="F1" library="RoboJackets-Fuses" package="F1206" value="3A" x="8.81" y="23.18" smashed="yes">
+<attribute name="NAME" x="6.81" y="24.68" size="1" layer="25"/>
+</element>
 </elements>
 <signals>
@@
 <wire x1="12.15" y1="31.35" x2="12.15" y2="30.2" width="0.2" layer="16"/>
 <wire x1="12.15" y1="30.2" x2="13" y2="29.35" width="0.2" layer="16"/>
-<wire x1="13" y1="29.35" x2="20.854975" y2="29.35" width="0.2" layer="16"/>
-<wire x1="20.854975" y1="29.35" x2="21.63" y2="28.574975" width="0.2" layer="16"/>
-<wire x1="23.47" y1="17.92" x2="23.47" y2="14.71" width="0.2" layer="16"/>
-<wire x1="23.47" y1="17.92" x2="21.63" y2="19.76" width="0.2" layer="16"/>
-<wire x1="21.63" y1="28.574975" x2="21.63" y2="19.76" width="0.2" layer="16"/>
+<wire x1="23.8292875" y1="15.0692875" x2="23.47" y2="14.71" width="0.2" layer="16"/>
+<via x="23.82" y="28.04" extent="1-16" drill="0.35"/>
+<wire x1="22.93218125" y1="29.37" x2="23.38781875" y2="29.37" width="0.2" layer="16"/>
+<wire x1="23.38781875" y1="29.37" x2="23.71" y2="29.04781875" width="0.2" layer="16"/>
+<wire x1="23.71" y1="28.15" x2="23.82" y2="28.04" width="0.2" layer="16"/>
+<wire x1="23.71" y1="29.04781875" x2="23.71" y2="28.15" width="0.2" layer="16"/>
+<wire x1="22.91218125" y1="29.35" x2="22.93218125" y2="29.37" width="0.2" layer="16"/>
+<wire x1="23.82" y1="28.04" x2="23.82" y2="22.0006625" width="0.2" layer="1"/>
+<wire x1="23.82" y1="22.0006625" x2="23.8292875" y2="21.991375" width="0.2" layer="1"/>
+<via x="23.8292875" y="21.991375" extent="1-16" drill="0.35"/>
+<wire x1="23.8292875" y1="21.991375" x2="23.8292875" y2="15.0692875" width="0.2" layer="16"/>
+<wire x1="13" y1="29.35" x2="22.91218125" y2="29.35" width="0.2" layer="16"/>
 </signal>
 <signal name="ENC_B">
@@
 <contactref element="U1" pad="10"/>
 <wire x1="9.61" y1="31.35" x2="9.61" y2="29.39" width="0.2" layer="16"/>
-<wire x1="9.61" y1="29.39" x2="10" y2="29" width="0.2" layer="16"/>
-<wire x1="10" y1="29" x2="20.27" y2="29" width="0.2" layer="16"/>
-<wire x1="21.03" y1="28.24" x2="21.03" y2="20.76" width="0.2" layer="16"/>
-<wire x1="21.03" y1="20.76" x2="18.39" y2="18.12" width="0.2" layer="16"/>
-<wire x1="18.39" y1="18.12" x2="18.39" y2="14.71" width="0.2" layer="16"/>
-<wire x1="20.27" y1="29" x2="21.03" y2="28.24" width="0.2" layer="16"/>
+<wire x1="9.61" y1="29.39" x2="10.03" y2="28.97" width="0.2" layer="16"/>
+<wire x1="23.3" y1="18.92" x2="19.09" y2="14.71" width="0.2" layer="16"/>
+<wire x1="18.39" y1="14.71" x2="19.09" y2="14.71" width="0.2" layer="16"/>
+<wire x1="23.01" y1="28.97" x2="23.16" y2="28.82" width="0.2" layer="16"/>
+<via x="23.16" y="28.82" extent="1-16" drill="0.35"/>
+<wire x1="23.16" y1="28.82" x2="23.16" y2="21.6" width="0.2" layer="1"/>
+<via x="23.16" y="21.6" extent="1-16" drill="0.35"/>
+<wire x1="23.16" y1="21.6" x2="23.3" y2="21.46" width="0.2" layer="16"/>
+<wire x1="23.3" y1="21.46" x2="23.3" y2="18.92" width="0.2" layer="16"/>
+<wire x1="10.03" y1="28.97" x2="23.01" y2="28.97" width="0.2" layer="16"/>
 </signal>
 <signal name="+5V">
@@
 <wire x1="9.37" y1="3.42" x2="12" y2="3.42" width="0.2" layer="16"/>
 <wire x1="6.08" y1="28.9" x2="4.95" y2="27.77" width="0.2" layer="16"/>
-<wire x1="4.95" y1="27.77" x2="4.95" y2="19.58" width="0.2" layer="16"/>
-<wire x1="7.18904375" y1="17.34095625" x2="4.95" y2="19.58" width="0.2" layer="16"/>
 <wire x1="7.18904375" y1="17.34095625" x2="7.48" y2="17.34095625" width="0.2" layer="16"/>
 <via x="7.57904375" y="17.34095625" extent="1-16" drill="0.35"/>
@@
 <wire x1="5.88" y1="16.79" x2="6.43095625" y2="17.34095625" width="0.2" layer="16"/>
 <wire x1="6.43095625" y1="17.34095625" x2="7.48" y2="17.34095625" width="0.2" layer="16"/>
+<contactref element="R6" pad="2"/>
+<wire x1="9.48" y1="10.45" x2="9.48" y2="8.34" width="0.2" layer="16"/>
+<wire x1="9.48" y1="8.34" x2="8.23" y2="7.09" width="0.2" layer="16"/>
+<wire x1="4.95" y1="27.77" x2="4.95" y2="23.38" width="0.2" layer="16"/>
+<wire x1="4.95" y1="23.38" x2="5.04" y2="23.29" width="0.2" layer="16"/>
+<via x="5.04" y="23.29" extent="1-16" drill="0.35"/>
+<wire x1="5.04" y1="23.29" x2="5.04" y2="19.43" width="0.2" layer="1"/>
+<wire x1="7.12904375" y1="17.34095625" x2="7.57904375" y2="17.34095625" width="0.2" layer="1"/>
+<wire x1="5.04" y1="19.43" x2="7.12904375" y2="17.34095625" width="0.2" layer="1"/>
 </signal>
 <signal name="GND">
@@
 </signal>
 <signal name="+12V">
-<contactref element="U2" pad="5"/>
-<contactref element="C4" pad="1"/>
-<contactref element="C3" pad="1"/>
 <contactref element="U3" pad="1"/>
 <contactref element="U3" pad="3"/>
 <contactref element="J1" pad="1"/>
 <contactref element="J2" pad="1"/>
-<wire x1="8.59" y1="28.15" x2="6.756" y2="28.15" width="0.8" layer="1"/>
-<wire x1="8.59" y1="28.15" x2="13.605" y2="23.135" width="0.8" layer="1"/>
-<wire x1="13.605" y1="23.135" x2="13.605" y2="22.3466" width="0.8" layer="1"/>
-<wire x1="13.605" y1="20.145" x2="13.605" y2="22.3466" width="0.8" layer="1"/>
 <wire x1="13.605" y1="20.145" x2="13.9" y2="19.85" width="0.8" layer="1"/>
 <wire x1="13.9" y1="19.85" x2="15.09" y2="18.66" width="0.8" layer="1"/>
-<wire x1="11.69" y1="21.11" x2="12.7" y2="21.11" width="0.8" layer="16"/>
-<wire x1="12.7" y1="21.11" x2="12.74" y2="21.15" width="0.4" layer="16"/>
-<via x="12.74" y="21.15" extent="1-16" drill="0.35"/>
-<wire x1="13.605" y1="22.3466" x2="12.74" y2="21.4816" width="0.8" layer="1"/>
-<wire x1="12.74" y1="21.15" x2="12.74" y2="21.4816" width="0.8" layer="1"/>
-<wire x1="11.74" y1="23.56" x2="11.74" y2="21.16" width="0.8" layer="16"/>
-<wire x1="11.74" y1="21.16" x2="11.69" y2="21.11" width="0.4" layer="16"/>
-<wire x1="6.756" y1="28.15" x2="3.676" y2="25.07" width="0.8" layer="1"/>
-<wire x1="3.676" y1="25.07" x2="3.28" y2="25.07" width="0.8" layer="1"/>
-<wire x1="3.28" y1="25.07" x2="3.02" y2="25.07" width="0.8" layer="1"/>
+<wire x1="3.02" y1="25.07" x2="3.28" y2="25.07" width="0.8" layer="1"/>
 <wire x1="15.09" y1="18.66" x2="21.7" y2="18.66" width="0.8" layer="1"/>
 <wire x1="27.92" y1="24.88" x2="27.92" y2="25.09" width="0.8" layer="1"/>
@@
 <wire x1="4.31" y1="24.04" x2="3.28" y2="25.07" width="0.2" layer="1"/>
 <wire x1="4.31" y1="15.83" x2="4.31" y2="24.04" width="0.2" layer="1"/>
+<contactref element="F1" pad="1"/>
+<wire x1="5.498" y1="25.07" x2="7.388" y2="23.18" width="0.8" layer="1"/>
+<wire x1="7.388" y1="23.18" x2="10.423" y2="20.145" width="0.8" layer="1"/>
+<wire x1="10.423" y1="20.145" x2="13.605" y2="20.145" width="0.8" layer="1"/>
+<wire x1="3.02" y1="25.07" x2="5.498" y2="25.07" width="0.8" layer="1"/>
 </signal>
 <signal name="IN2">
@@
 <wire x1="4.65" y1="5.76" x2="4.34" y2="6.07" width="0.2" layer="1"/>
 <wire x1="14.52" y1="5.76" x2="4.65" y2="5.76" width="0.2" layer="1"/>
+<contactref element="R6" pad="1"/>
+<wire x1="7.78" y1="10.45" x2="7.78" y2="9.51" width="0.2" layer="16"/>
+<wire x1="7.78" y1="9.51" x2="4.34" y2="6.07" width="0.2" layer="16"/>
+</signal>
+<signal name="12V_FUSE">
+<contactref element="U2" pad="5"/>
+<contactref element="C4" pad="1"/>
+<contactref element="C3" pad="1"/>
+<wire x1="11.69" y1="21.11" x2="12.7" y2="21.11" width="0.8" layer="16"/>
+<wire x1="12.7" y1="21.11" x2="12.74" y2="21.15" width="0.4" layer="16"/>
+<via x="12.74" y="21.15" extent="1-16" drill="0.35"/>
+<wire x1="13.605" y1="22.3466" x2="12.74" y2="21.4816" width="0.8" layer="1"/>
+<wire x1="12.74" y1="21.15" x2="12.74" y2="21.4816" width="0.8" layer="1"/>
+<wire x1="11.74" y1="23.56" x2="11.74" y2="21.16" width="0.8" layer="16"/>
+<wire x1="11.74" y1="21.16" x2="11.69" y2="21.11" width="0.4" layer="16"/>
+<contactref element="F1" pad="2"/>
+<wire x1="10.232" y1="23.18" x2="12.7716" y2="23.18" width="0.8" layer="1"/>
+<wire x1="12.7716" y1="23.18" x2="13.605" y2="22.3466" width="0.8" layer="1"/>
 </signal>
 </signals>

Commit message: Exported files for Version 1.0
Parts:
- added C7: 1uF, rcl:C0603
- added C8, C9: 0.1u, rcl:C0603
- C4: value 1u -> 10u
- C5: value 2.2u -> 100p
- C6: value 0.1u -> 2.2u
- moved J3 1.38 mm to (10.6, 3.42)
- moved F1 0.55 mm to (9.36, 23.2)
Connections:
- net +12V: now also C7.1, C8.1
- net GND: now also C7.2, C8.2, C9.2
- net RST: now also C9.1
Routing:
- net +12V: track 48.4 -> 52.5 mm
- net RST: track 18.0 -> 20.6 mm
- net +5V: track 60.5 -> 59.1 mm
- net ZERO: track 11.8 -> 12.4 mm
- net 12V_FUSE: track 8.81 -> 8.26 mm
- net ENC_A: track 27.7 -> 28.3 mm
Other:
- board text added: "M+"
- board text added: "ZERO"
