File: drive_ctrl.sch (EAGLE design)
At the start: 24 parts, among them J1 4-PIN_2MM-V, J2 4-PIN_2MM-V, J3 ZEROING_SENSOR, U1 ATTINY84ATTINY84-20PU, U2 DRV8871HSOP-8, U3 AP2210-5KSOT-23-5

Commit message: Added fuse, decoupling capacitors, and changed routing
Parts:
- added F1: 3A, RoboJackets-Fuses:CHIP_FUSE1206
- added R6: 1k, rcl:R-US_R0603
Connections:
- new net 12V_FUSE: C3.1, C4.1, F1.2, U2.VM
- net +12V: now also F1.1; no longer C3.1, C4.1, U2.VM
- net +5V: now also R6.2
- net RST: now also R6.1
Other:
- note added: "Jumper and pull-up for on-board reset"
- moved on the sheet: C1, C2, C3, C4, C5, C6, J1, J2, J3, JP2, R1, U1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

Commit message: Exported files for Version 1.0
Parts:
- added C7: 1uF, rcl:C-USC0603
- added C8, C9: 0.1u, rcl:C-USC0603
- C4: value 1u -> 10u
- C5: value 2.2u -> 100p
- C6: value 0.1u -> 2.2u
Connections:
- net +12V: now also C7.1, C8.1
- net GND: now also C7.2, C8.2, C9.2
- net RST: now also C9.1
Other:
- note added: "Detects if wheel is at a 0 position by detecting embedded magnet"
- note added: "NOTE: All capacitors rated 25V or more"
- moved on the sheet: J3, JP1, JP2
